Commit message: intento con moveit_4

File: scara_ws/src/scada_urdf/urdf/scada_urdf (copy).urdf (robot description, URDF)
Before this commit: robot scada_urdf, 5 links, 4 joints
Links:
- added link world
Joints:
- added joint dummy_joint: type fixed, parent world, child base_link, origin xyz=0 0 0 rpy=0 0 0

File: scara_ws/src/scada_urdf/urdf/scada_urdf_moveit.urdf (robot description, URDF)
Before this commit: robot scada_urdf, 6 links, 5 joints
Links:
- removed link world
Joints:
- removed joint dummy_joint
