Commit message: gitignore

File: scara_ws/src/scada_urdf/urdf/scada_urdf.urdf (robot description, URDF)
Before this commit: robot scada_urdf, 5 links, 4 joints
Links:
- removed link base
- added link base_link, mass 25.2913216476849; collision mesh filename=package://scada_urdf/meshes/base.STL; visual mesh filename=package://scada_urdf/meshes/base.STL
Joints:
- joint hombro: parent base -> base_link
- joint muneca: limit lower=0 upper=0 effort=0 velocity=0 -> lower=-1 upper=1 effort=0 velocity=1

Commit message: conexion exitosa con gazebo

File: scara_ws/src/scada_urdf/urdf/scada_urdf.urdf (robot description, URDF)
Before this commit: robot scada_urdf, 6 links, 5 joints
Joints:
- joint muneca: limit lower=-1 upper=1 effort=0 velocity=1 -> lower=-1 upper=1 effort=1 velocity=1

Commit message: conexion exitosa con gazebo

File: scara_ws/src/scada_urdf/urdf/scada_urdf.urdf (robot description, URDF)
Before this commit: robot scada_urdf, 6 links, 5 joints
Joints:
- joint muneca: limit lower=-1 upper=1 effort=1 velocity=1 -> (none); type prismatic -> fixed

Commit message: conexion exitosa con gazebo

File: scara_ws/src/scada_urdf/urdf/scada_urdf.urdf (robot description, URDF)
Before this commit: robot scada_urdf, 6 links, 5 joints
Joints:
- joint muneca: limit (none) -> lower=-1 upper=1 effort=1 velocity=1; type fixed -> prismatic
