Commit message: Correccion

File: servo/servo_urdf/servo_urdf/urdf/servo_urdf.urdf (robot description, URDF)
Before this commit: robot servo_urdf, 2 links, 1 joints
Links:
- link puntero: mass 0.00088335655680429 -> 0.000883356556804291
Joints:
- joint junta: origin xyz=0.0174058777578102 0.006 0.0295 rpy=0 0 0 -> xyz=0.017406 0.006 0.0295 rpy=0 0 0
