Commit message: calibracion del robot

File: scara_ws/src/epson/urdf/epson.urdf (robot description, URDF)
Before this commit: robot epson, 6 links, 5 joints
Joints:
- joint articulacion: child dedo -> mano; limit (none) -> lower=0 upper=0.15 effort=80 velocity=1; origin xyz=0 0 0 rpy=0 0 0 -> xyz=0.37763 0 0.020231 rpy=0 0 0; parent mano -> brazo; type continuous -> prismatic
- joint codo: origin xyz=0.4025 0 0 rpy=0 0 2.4099 -> xyz=0.4025 0 0 rpy=0 0 0
- joint hombro: origin xyz=0 0 0.5925 rpy=0 0 0.55607 -> xyz=0 0 0.5925 rpy=0 0 0
- joint muneca: child mano -> dedo; limit lower=0 upper=0.20 effort=80 velocity=1 -> (none); origin xyz=0.37763 0 0.020231 rpy=0 0 0 -> xyz=0 0 0 rpy=0 0 0; parent brazo -> mano; type prismatic -> continuous
